File: pcb/4by3.sch (KiCad schematic (older format))
At the start: 26 parts, among them K1 KEYSW, K10 KEYSW, K11 KEYSW, K12 KEYSW, K2 KEYSW, K3 KEYSW, K4 KEYSW, K5 KEYSW, K6 KEYSW, K7 KEYSW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

Commit message: Added images, created a pretty library
Parts:
- D1, D10, D11, D12, D2, D3, D4, D5, D6, D7, D8, D9: footprint Diodes_THT:D_DO-35_SOD27_P7.62mm_Horizontal -> 4by3:DIODE
- K1, K10, K11, K12, K2, K3, K4, K5, K6, K7, K8, K9: footprint Keyboard:CHERRY_PCB_100H -> 4by3:CHERRY_MX_PCB
- M1: footprint SparkFun-Boards:ARDUINO_PRO_MICRO -> 4by3:PRO_MICRO
- SW1: footprint Sparkfun_Switches:TACTILE_SWITCH_SMD_5.2MM -> 4by3:RESET_BUTTON
Changed lines of the file:
@@
 LIBS:valves
 LIBS:keyboard_parts
-LIBS:mkl27z256vfm4
 LIBS:arduino_micro_shield
 LIBS:4xxx
@@
 LIBS:Teensy_3_and_LC_Series_Boards_v1.1
 LIBS:User-Submitted
+LIBS:4by3-cache
 EELAYER 25 0
 EELAYER END
@@
 F 0 "K3" H 1300 4700 60  0000 C CNN
 F 1 "KEYSW" H 1350 4600 60  0001 C CNN
-F 2 "Keyboard:CHERRY_PCB_100H" H 1350 4700 60  0001 C CNN
+F 2 "4by3:CHERRY_MX_PCB" H 1350 4700 60  0001 C CNN
 F 3 "" H 1350 4700 60  0000 C CNN
 	1    1350 4700
@@
 F 0 "K2" H 1300 3700 60  0000 C CNN
 F 1 "KEYSW" H 1350 3600 60  0001 C CNN
-F 2 "Keyboard:CHERRY_PCB_100H" H 1350 3700 60  0001 C CNN
+F 2 "4by3:CHERRY_MX_PCB" H 1350 3700 60  0001 C CNN
 F 3 "" H 1350 3700 60  0000 C CNN
 	1    1350 3700
@@
 F 0 "K1" H 1300 2700 60  0000 C CNN
 F 1 "KEYSW" H 1350 2600 60  0001 C CNN
-F 2 "Keyboard:CHERRY_PCB_100H" H 1350 2700 60  0001 C CNN
+F 2 "4by3:CHERRY_MX_PCB" H 1350 2700 60  0001 C CNN
 F 3 "" H 1350 2700 60  0000 C CNN
 	1    1350 2700
@@
 F 0 "D1" H 950 3050 50  0000 C CNN
 F 1 "D" H 950 2850 50  0000 C CNN
-F 2 "Diodes_THT:D_DO-35_SOD27_P7.62mm_Horizontal" H 950 2950 50  0001 C CNN
+F 2 "4by3:DIODE" H 950 2950 50  0001 C CNN
 F 3 "" H 950 2950 50  0001 C CNN
 	1    950  2950
@@
 F 0 "D2" H 950 4050 50  0000 C CNN
 F 1 "D" H 950 3850 50  0000 C CNN
-F 2 "Diodes_THT:D_DO-35_SOD27_P7.62mm_Horizontal" H 950 3950 50  0001 C CNN
+F 2 "4by3:DIODE" H 950 3950 50  0001 C CNN
 F 3 "" H 950 3950 50  0001 C CNN
 	1    950  3950
@@
 F 0 "D3" H 950 5050 50  0000 C CNN
 F 1 "D" H 950 4850 50  0000 C CNN
-F 2 "Diodes_THT:D_DO-35_SOD27_P7.62mm_Horizontal" H 950 4950 50  0001 C CNN
+F 2 "4by3:DIODE" H 950 4950 50  0001 C CNN
 F 3 "" H 950 4950 50  0001 C CNN
 	1    950  4950
@@
 F 0 "K6" H 2500 4700 60  0000 C CNN
 F 1 "KEYSW" H 2550 4600 60  0001 C CNN
-F 2 "Keyboard:CHERRY_PCB_100H" H 2550 4700 60  0001 C CNN
+F 2 "4by3:CHERRY_MX_PCB" H 2550 4700 60  0001 C CNN
 F 3 "" H 2550 4700 60  0000 C CNN
 	1    2550 4700
@@
 F 0 "K5" H 2500 3700 60  0000 C CNN
 F 1 "KEYSW" H 2550 3600 60  0001 C CNN
-F 2 "Keyboard:CHERRY_PCB_100H" H 2550 3700 60  0001 C CNN
+F 2 "4by3:CHERRY_MX_PCB" H 2550 3700 60  0001 C CNN
 F 3 "" H 2550 3700 60  0000 C CNN
 	1    2550 3700
@@
 F 0 "K4" H 2500 2700 60  0000 C CNN
 F 1 "KEYSW" H 2550 2600 60  0001 C CNN
-F 2 "Keyboard:CHERRY_PCB_100H" H 2550 2700 60  0001 C CNN
+F 2 "4by3:CHERRY_MX_PCB" H 2550 2700 60  0001 C CNN
 F 3 "" H 2550 2700 60  0000 C CNN
 	1    2550 2700
@@
 F 0 "D4" H 2150 3050 50  0000 C CNN
 F 1 "D" H 2150 2850 50  0000 C CNN
-F 2 "Diodes_THT:D_DO-35_SOD27_P7.62mm_Horizontal" H 2150 2950 50  0001 C CNN
+F 2 "4by3:DIODE" H 2150 2950 50  0001 C CNN
 F 3 "" H 2150 2950 50  0001 C CNN
 	1    2150 2950
@@
 F 0 "D5" H 2150 4050 50  0000 C CNN
 F 1 "D" H 2150 3850 50  0000 C CNN
-F 2 "Diodes_THT:D_DO-35_SOD27_P7.62mm_Horizontal" H 2150 3950 50  0001 C CNN
+F 2 "4by3:DIODE" H 2150 3950 50  0001 C CNN
 F 3 "" H 2150 3950 50  0001 C CNN
 	1    2150 3950
@@
 F 0 "D6" H 2150 5050 50  0000 C CNN
 F 1 "D" H 2150 4850 50  0000 C CNN
-F 2 "Diodes_THT:D_DO-35_SOD27_P7.62mm_Horizontal" H 2150 4950 50  0001 C CNN
+F 2 "4by3:DIODE" H 2150 4950 50  0001 C CNN
 F 3 "" H 2150 4950 50  0001 C CNN
 	1    2150 4950
@@
 F 0 "K9" H 3700 4700 60  0000 C CNN
 F 1 "KEYSW" H 3750 4600 60  0001 C CNN
-F 2 "Keyboard:CHERRY_PCB_100H" H 3750 4700 60  0001 C CNN
+F 2 "4by3:CHERRY_MX_PCB" H 3750 4700 60  0001 C CNN
 F 3 "" H 3750 4700 60  0000 C CNN
 	1    3750 4700
@@
 F 0 "K8" H 3700 3700 60  0000 C CNN
 F 1 "KEYSW" H 3750 3600 60  0001 C CNN
-F 2 "Keyboard:CHERRY_PCB_100H" H 3750 3700 60  0001 C CNN
+F 2 "4by3:CHERRY_MX_PCB" H 3750 3700 60  0001 C CNN
 F 3 "" H 3750 3700 60  0000 C CNN
 	1    3750 3700
@@
 F 0 "K7" H 3700 2700 60  0000 C CNN
 F 1 "KEYSW" H 3750 2600 60  0001 C CNN
-F 2 "Keyboard:CHERRY_PCB_100H" H 3750 2700 60  0001 C CNN
+F 2 "4by3:CHERRY_MX_PCB" H 3750 2700 60  0001 C CNN
 F 3 "" H 3750 2700 60  0000 C CNN
 	1    3750 2700
@@
 F 0 "D7" H 3350 3050 50  0000 C CNN
 F 1 "D" H 3350 2850 50  0000 C CNN
-F 2 "Diodes_THT:D_DO-35_SOD27_P7.62mm_Horizontal" H 3350 2950 50  0001 C CNN
+F 2 "4by3:DIODE" H 3350 2950 50  0001 C CNN
 F 3 "" H 3350 2950 50  0001 C CNN
 	1    3350 2950
@@
 F 0 "D8" H 3350 4050 50  0000 C CNN
 F 1 "D" H 3350 3850 50  0000 C CNN
-F 2 "Diodes_THT:D_DO-35_SOD27_P7.62mm_Horizontal" H 3350 3950 50  0001 C CNN
+F 2 "4by3:DIODE" H 3350 3950 50  0001 C CNN
 F 3 "" H 3350 3950 50  0001 C CNN
 	1    3350 3950
@@
 F 0 "D9" H 3350 5050 50  0000 C CNN
 F 1 "D" H 3350 4850 50  0000 C CNN
-F 2 "Diodes_THT:D_DO-35_SOD27_P7.62mm_Horizontal" H 3350 4950 50  0001 C CNN
+F 2 "4by3:DIODE" H 3350 4950 50  0001 C CNN
 F 3 "" H 3350 4950 50  0001 C CNN
 	1    3350 4950
@@
 F 0 "K12" H 4900 4700 60  0000 C CNN
 F 1 "KEYSW" H 4950 4600 60  0001 C CNN
-F 2 "Keyboard:CHERRY_PCB_100H" H 4950 4700 60  0001 C CNN
+F 2 "4by3:CHERRY_MX_PCB" H 4950 4700 60  0001 C CNN
 F 3 "" H 4950 4700 60  0000 C CNN
 	1    4950 4700
@@
 F 0 "K11" H 4900 3700 60  0000 C CNN
 F 1 "KEYSW" H 4950 3600 60  0001 C CNN
-F 2 "Keyboard:CHERRY_PCB_100H" H 4950 3700 60  0001 C CNN
+F 2 "4by3:CHERRY_MX_PCB" H 4950 3700 60  0001 C CNN
 F 3 "" H 4950 3700 60  0000 C CNN
 	1    4950 3700
@@
 F 0 "K10" H 4900 2700 60  0000 C CNN
 F 1 "KEYSW" H 4950 2600 60  0001 C CNN
-F 2 "Keyboard:CHERRY_PCB_100H" H 4950 2700 60  0001 C CNN
+F 2 "4by3:CHERRY_MX_PCB" H 4950 2700 60  0001 C CNN
 F 3 "" H 4950 2700 60  0000 C CNN
 	1    4950 2700
@@
 F 0 "D10" H 4550 3050 50  0000 C CNN
 F 1 "D" H 4550 2850 50  0000 C CNN
-F 2 "Diodes_THT:D_DO-35_SOD27_P7.62mm_Horizontal" H 4550 2950 50  0001 C CNN
+F 2 "4by3:DIODE" H 4550 2950 50  0001 C CNN
 F 3 "" H 4550 2950 50  0001 C CNN
 	1    4550 2950
@@
 F 0 "D11" H 4550 4050 50  0000 C CNN
 F 1 "D" H 4550 3850 50  0000 C CNN
-F 2 "Diodes_THT:D_DO-35_SOD27_P7.62mm_Horizontal" H 4550 3950 50  0001 C CNN
+F 2 "4by3:DIODE" H 4550 3950 50  0001 C CNN
 F 3 "" H 4550 3950 50  0001 C CNN
 	1    4550 3950
@@
 F 0 "D12" H 4550 5050 50  0000 C CNN
 F 1 "D" H 4550 4850 50  0000 C CNN
-F 2 "Diodes_THT:D_DO-35_SOD27_P7.62mm_Horizontal" H 4550 4950 50  0001 C CNN
+F 2 "4by3:DIODE" H 4550 4950 50  0001 C CNN
 F 3 "" H 4550 4950 50  0001 C CNN
 	1    4550 4950
@@
 F 0 "M1" H 1050 2100 50  0000 C CNN
 F 1 "PRO_MICRO" H 1500 2100 50  0000 C CNN
-F 2 "SparkFun-Boards:ARDUINO_PRO_MICRO" H 1330 1500 20  0001 C CNN
+F 2 "4by3:PRO_MICRO" H 1330 1500 20  0001 C CNN
 F 3 "" H 1300 1350 60  0001 C CNN
 	1    1300 1350
@@
 F 0 "SW1" H 2950 700 50  0000 C TNN
 F 1 "SW_PUSH" H 2950 850 50  0000 C BNN
-F 2 "Sparkfun_Switches:TACTILE_SWITCH_SMD_5.2MM" H 2950 750 60  0001 C CNN
+F 2 "4by3:RESET_BUTTON" H 2950 750 60  0001 C CNN
 F 3 "" H 2950 750 60  0000 C CNN
 	1    2950 750
